File: PSFB_PCB/PSFB.kicad_pcb (KiCad board)
At the start: 4 copper layers, 182.2 x 127.5 mm, 128 parts, among them IC1 TMCS1133B7AQDVGR, IC10 ISOUSB111DWXR, IC12 TPSI3050DWZR, IC13 OPA365AIDBVTG4, IC2 HCNR201-300E, IC3 OPA365AIDBVTG4, IC4 UA78M05CDCYG3, IC5 SN74LVC1G08DBVR, IC6 TLV1702AIDGK, IC7 OPA2376AQDRQ1, IC9 TMCS1133B7AQDVGR, J1 12V_Jumper_for_5V, J23 VOUT_CHARGER, J24 5V_PIN_IN_DEBUG, J3 JUMPER_BOOT, J5 STLINK_PIN, J6 USB_C, Q1 R6086YNZ4C13, Q2 R6086YNZ4C13, U1 STM32G474CBTx, U2 MASTERGAN6TR, U3 SN6507DGQ, U4 MASTERGAN6TR, U5 ACPL-M61L-000E

Commit message: updating Work
Parts:
- added C32: 10u, Capacitor_SMD:C_1206_3216Metric, F.Cu at (33.2, 86.4)
- added C50: 25V 0.1uF X7R, Capacitor_SMD:C_0805_2012Metric_Pad1.18x1.45mm_HandSolder, F.Cu at (36.0, 92.4)
- added C51: 6.3V 47uF X7S, Capacitor_SMD:C_1206_3216Metric_Pad1.33x1.80mm_HandSolder, F.Cu at (47.0, 85.2)
- added C54: 270u, Capacitor_THT:CP_Radial_D25.0mm_P10.00mm_SnapIn, F.Cu at (50.2, 55.4)
- added C56: 10u, Capacitor_SMD:C_1206_3216Metric, F.Cu at (33.2, 88.8)
- added D10: LED RED, LED_SMD:LED_1206_3216Metric_Pad1.42x1.75mm_HandSolder, F.Cu at (42.8, 37.2)
- added D11: LED AMBAR, LED_SMD:LED_1206_3216Metric_Pad1.42x1.75mm_HandSolder, F.Cu at (45.2, 37.2)
- added D12: ESD441DPLR, oscar:ESD441DPLR, F.Cu at (47.6, -0.47)
- added D13: ESD441DPLR, oscar:ESD441DPLR, F.Cu at (47.6, 2.94)
- added D14: LED GREEN, LED_SMD:LED_0603_1608Metric, F.Cu at (36.4, 37.0)
- added D15: LED GREEN, LED_SMD:LED_0603_1608Metric, F.Cu at (38.0, 37.0)
- added D7: LED GREEN, LED_SMD:LED_0603_1608Metric, F.Cu at (53.2, 37.2)
- added D8: LED GREEN, LED_SMD:LED_0603_1608Metric, F.Cu at (51.6, 37.2)
- added D9: LED GREEN, LED_SMD:LED_0603_1608Metric, F.Cu at (50.0, 37.2)
- added J10: V_IN_SENSE, Connector_PinHeader_2.54mm:PinHeader_1x01_P2.54mm_Vertical, F.Cu at (34.2, -8.26)
- added J11: I_OUT_SENSE, Connector_PinHeader_2.54mm:PinHeader_1x01_P2.54mm_Vertical, F.Cu at (34.2, -3.67)
- added J12: V_OUT_SENSE, Connector_PinHeader_2.54mm:PinHeader_1x01_P2.54mm_Vertical, F.Cu at (34.2, 0.92)
- added J13: V_BAT_SENSE, Connector_PinHeader_2.54mm:PinHeader_1x01_P2.54mm_Vertical, F.Cu at (38.8, -17.4)
- added J14: GND_SENSE, Connector_PinHeader_2.54mm:PinHeader_1x01_P2.54mm_Vertical, F.Cu at (38.8, -12.8)
- added J15: CTRL_AH, Connector_PinHeader_2.54mm:PinHeader_1x01_P2.54mm_Vertical, F.Cu at (38.8, -8.26)
- added J16: CTRL_AL, Connector_PinHeader_2.54mm:PinHeader_1x01_P2.54mm_Vertical, F.Cu at (38.8, -3.67)
- added J17: CTRL_BL, Connector_PinHeader_2.54mm:PinHeader_1x01_P2.54mm_Vertical, F.Cu at (38.8, 0.92)
- added J18: CTRL_BH, Connector_PinHeader_2.54mm:PinHeader_1x01_P2.54mm_Vertical, F.Cu at (43.4, -17.4)
- added J19: HVDC_POWER_IN, oscar:1731734, F.Cu at (23.4, 134.6)
- added J2: GND_S, Connector_PinHeader_2.54mm:PinHeader_1x01_P2.54mm_Vertical, F.Cu at (34.2, -17.4)
- added J20: 5VCC_S, Connector_PinHeader_2.54mm:PinHeader_1x01_P2.54mm_Vertical, F.Cu at (43.4, -12.8)
- added J21: Vref_S, Connector_PinHeader_2.54mm:PinHeader_1x01_P2.54mm_Vertical, F.Cu at (43.4, -8.26)
- added J22: VDC_S_SENSE_S, Connector_PinHeader_2.54mm:PinHeader_1x01_P2.54mm_Vertical, F.Cu at (43.4, -3.67)
- added J4: 3.3V_PIN_IN_DEBUG, Connector_PinHeader_2.54mm:PinHeader_1x02_P2.54mm_Vertical, F.Cu at (52.2, 83.6)
- added J7: Power_Terminal_12V, oscar:15465512, F.Cu at (24.9, 58.9)
- added J8: 12V_Jumper_for_3.3V, Connector_PinHeader_2.54mm:PinHeader_1x02_P2.54mm_Vertical, F.Cu at (31.7, 71.3)
- added J9: I_IN_SENSE, Connector_PinHeader_2.54mm:PinHeader_1x01_P2.54mm_Vertical, F.Cu at (34.2, -12.8)
- added L2: 3.3uH 70mOhm, oscar:784777033, F.Cu at (40.6, 83.6)
- added PS1: TPS561208DDCT, oscar:SOT95P280X110-6N, F.Cu at (33.2, 92.2)
- added R22: 180k, Resistor_SMD:R_0603_1608Metric_Pad0.98x0.95mm_HandSolder, F.Cu at (34.1, 7.89)
- added R23: 1.3k, Resistor_SMD:R_0603_1608Metric_Pad0.98x0.95mm_HandSolder, F.Cu at (34.1, 10.4)
- added R26: 150, Resistor_SMD:R_0603_1608Metric_Pad0.98x0.95mm_HandSolder, F.Cu at (53.2, 40.4)
- added R27: 150, Resistor_SMD:R_0603_1608Metric_Pad0.98x0.95mm_HandSolder, F.Cu at (51.6, 40.4)
- added R28: 150, Resistor_SMD:R_0603_1608Metric_Pad0.98x0.95mm_HandSolder, F.Cu at (50.0, 40.4)
- added R29: 270, Resistor_SMD:R_0603_1608Metric_Pad0.98x0.95mm_HandSolder, F.Cu at (42.8, 41.4)
- added R30: 270, Resistor_SMD:R_0603_1608Metric_Pad0.98x0.95mm_HandSolder, F.Cu at (45.2, 41.4)
- added R33: 100k, Resistor_SMD:R_1206_3216Metric_Pad1.30x1.75mm_HandSolder, F.Cu at (32.6, 113.6)
- added R34: 100k, Resistor_SMD:R_1206_3216Metric_Pad1.30x1.75mm_HandSolder, F.Cu at (32.6, 108.7)
- added R35: 100k, Resistor_SMD:R_1206_3216Metric_Pad1.30x1.75mm_HandSolder, F.Cu at (32.6, 103.7)
- added R40: 33k, Resistor_SMD:R_0603_1608Metric_Pad0.98x0.95mm_HandSolder, F.Cu at (33.2, 97.6)
- added R42: 1.8k, Resistor_SMD:R_0603_1608Metric_Pad0.98x0.95mm_HandSolder, F.Cu at (36.4, 40.2)
- added R43: 150, Resistor_SMD:R_0603_1608Metric_Pad0.98x0.95mm_HandSolder, F.Cu at (38.0, 40.2)
- added R61: 10k, Resistor_SMD:R_0603_1608Metric_Pad0.98x0.95mm_HandSolder, F.Cu at (33.2, 96.0)
- added T1: MAIN TRANSFORMER, oscar:TRANSFORMER_PQ_PSFB, F.Cu at (145.7, 124.2)
- moved C11 125.3 mm to (75.2, 118.2), turned to 90 degrees
- moved C12 120.4 mm to (75.2, 135.6), turned to -90 degrees
- moved C10 112.0 mm to (48.2, 118.2), turned to 90 degrees
- moved C14 99.5 mm to (48.2, 135.7), turned to -90 degrees
- moved C1 23.8 mm to (114.0, 69.8)
- moved C2 23.8 mm to (104.8, 68.3)
- moved C3 23.8 mm to (104.2, 65.9)
- moved C4 23.8 mm to (102.7, 65.9)
- moved R24 23.8 mm to (118.0, 62.2)
- moved C5 23.8 mm to (115.5, 60.5)
- moved U1 23.8 mm to (110.2, 64.4)
- moved J3 23.8 mm to (120.6, 63.1)
- moved C44 21.1 mm to (88.3, 47.3)
- moved C45 21.1 mm to (83.3, 47.3)
- moved C47 21.1 mm to (86.2, 63.8)
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Routing:
- net 12Vcc: track 16.8 -> 248.1 mm, vias 0 -> 2
- net 3.3Vcc: track 50.0 -> 202.0 mm
- net EN: track 0.00 -> 25.5 mm, vias 0 -> 2
- net Net-(IC12-VDRV): track 52.8 -> 35.7 mm
- net MOS_S: track 23.4 -> 39.5 mm
- net SW: track 0.00 -> 15.6 mm, vias 0 -> 3
- net VDC_S: track 23.0 -> 12.9 mm
- net Net-(PS1-VFB): track 0.00 -> 4.97 mm
- net CTRLB_H: track 8.93 -> 4.11 mm
- net CTRLB_L: track 8.57 -> 4.13 mm
- net Net-(PS1-VBST): track 0.00 -> 4.07 mm
- net Net-(R34-Pad2): track 0.00 -> 1.90 mm
- net Net-(R33-Pad2): track 0.00 -> 1.85 mm
- net Net-(J1-Pin_1): track 22.5 -> 21.4 mm
- net 5Vcc: track 152.4 -> 153.0 mm, vias 4 -> 5
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- added copper zone on B.Cu, net GND_USB
- added copper zone on F.Cu, net GND_USB
- added copper zone on In1.Cu, net GND_USB
- added copper zone on In2.Cu, net GND_USB
- added copper zone on F.Cu, net HVDC+
- added copper zone on F.Cu, net VDC_S
- added copper zone on F.Cu, net VOUT-
- added copper zone on F.Cu, net transformer_P_A
- added copper zone on F.Cu, net transformer_S_N
- added copper zone on F.Cu, net transformer_S_P
Other:
- board size 182.2 x 127.5 mm -> 387.2 x 127.5 mm

Commit message: MCU conections
Parts:
- C25: moved to F.Cu
- moved R22 131.3 mm to (121.5, 105.9), turned to 90 degrees
- moved R23 126.0 mm to (119.0, 103.5), turned to 180 degrees
- moved D10 84.6 mm to (126.0, 52.4)
- moved R29 84.6 mm to (126.0, 56.6)
- moved D7 82.3 mm to (134.1, 52.4)
- moved R26 82.3 mm to (134.1, 55.6)
- moved D8 82.3 mm to (132.4, 52.4)
- moved D9 82.3 mm to (130.8, 52.4)
- moved R27 82.3 mm to (132.4, 55.6)
- moved R28 82.3 mm to (130.8, 55.6)
- moved D11 79.9 mm to (123.7, 52.4)
- moved R30 79.9 mm to (123.7, 56.6)
- moved R42 76.9 mm to (111.8, 55.6)
- moved D14 76.9 mm to (111.8, 52.4)
- moved D15 76.9 mm to (113.3, 52.4)
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Connections:
- U1 pad 10: unconnected-(U1-PA2-Pad10) -> LED_MCU_ON
- U1 pad 11: unconnected-(U1-PA3-Pad11) -> LED_OK
- U1 pad 12: unconnected-(U1-PA4-Pad12) -> LED_STATUS
- U1 pad 13: unconnected-(U1-PA5-Pad13) -> LED_FAULT_MCU
- U1 pad 14: unconnected-(U1-PA6-Pad14) -> LED_FAULT_BATTERY
- U1 pad 16: I_IN_SENSE -> I_OUT_SENSE
- U1 pad 17: LED_MCU_ON -> unconnected-(U1-PB1-Pad17)
- U1 pad 18: LED_OK -> unconnected-(U1-PB2-Pad18)
- U1 pad 28: VDC_S_SENSE -> CTRLA_L
- U1 pad 29: V_BAT_FLAG -> CTRLA_H
- U1 pad 30: CTRLA_L -> unconnected-(U1-PA8-Pad30)
- U1 pad 31: CTRLA_H -> I_IN_SENSE
- U1 pad 40: LED_STATUS -> unconnected-(U1-PB3-Pad40)
- U1 pad 41: LED_FAULT_MCU -> unconnected-(U1-PB4-Pad41)
- U1 pad 42: LED_FAULT_BATTERY -> unconnected-(U1-PB5-Pad42)
- U1 pad 43: SSR -> unconnected-(U1-PB6-Pad43)
- U1 pad 5: unconnected-(U1-PF0-Pad5) -> VDC_P_SENSE
- U1 pad 6: unconnected-(U1-PF1-Pad6) -> VDC_S_SENSE
- U1 pad 8: VDC_P_SENSE -> SSR
- U1 pad 9: I_OUT_SENSE -> V_BAT_FLAG
Routing:
- net 12Vcc: track 248.1 -> 90.7 mm
- net CTRLB_L: track 4.13 -> 112.3 mm
- net CTRLB_H: track 4.11 -> 110.5 mm
- net CTRLA_L: track 4.13 -> 93.3 mm
- net CTRLA_H: track 4.11 -> 91.6 mm
- net I_OUT_SENSE: track 0.00 -> 61.5 mm
- net 3.3Vcc: track 202.0 -> 144.9 mm, vias 3 -> 2
- net USB_DD_P: track 0.00 -> 41.0 mm, vias 0 -> 2
- net VDC_P_SENSE: track 0.00 -> 40.7 mm
- net USB_DD_N: track 0.00 -> 40.3 mm, vias 0 -> 2
- net I_IN_SENSE: track 0.00 -> 38.9 mm
- net NRST: track 7.35 -> 35.4 mm, vias 0 -> 1
- net SSR: track 0.00 -> 23.2 mm
- net VDC_S_SENSE: track 4.27 -> 26.2 mm
- net LED_MCU_ON: track 0.00 -> 19.8 mm
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