File: PSFB_PCB/PSFB.kicad_sch (KiCad schematic)
At the start: 54 parts, among them IC10 ISOUSB111DWXR, J10 V_IN_SENSE, J11 I_OUT_SENSE, J12 V_OUT_SENSE, J13 V_BAT_SENSE, J14 GND_SENSE, J15 CTRL_AH, J16 CTRL_AL, J17 CTRL_BL, J18 CTRL_BH, J2 GND_S, J20 5VCC_S, J21 Vref_S, J22 VDC_S_SENSE_S, J3 JUMPER_BOOT, J5 STLINK_PIN, J6 USB_C, J9 I_IN_SENSE, U1 STM32G474CBTx

Commit message: updating Work
Parts:
- removed TR1: Our Transformer, Transformer_THT:Transformer_Breve_TEZ-28x33, symbol Transformer:TEZ2.0-D-1
- added T1: MAIN TRANSFORMER, oscar:TRANSFORMER_PQ_PSFB, symbol Transformer:ED8_4
Connections:
- net transformer_P_B: now also T1.2
- net transformer_S_N: now also T1.3
- net at C29.2: now also T1.1
- new net transformer_S_P: T1.4
Other:
- moved on the sheet: C29
Changed lines of the file:
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@@
 	(wire
 		(pts
-			(xy 180.975 52.07) (xy 188.595 52.07)
+			(xy 180.975 52.07) (xy 189.23 52.07)
 		)
 		(stroke
@@
 	(global_label "transformer_P_A"
 		(shape input)
-		(at 180.975 41.91 180)
+		(at 181.61 41.91 180)
 		(fields_autoplaced yes)
 		(effects
@@
 		)
 		(property "Intersheetrefs" "${INTERSHEET_REFS}"
-			(at 162.629 41.91 0)
+			(at 163.264 41.91 0)
 			(effects
 				(font
@@
 	(global_label "transformer_S_N"
 		(shape output)
-		(at 198.755 52.07 0)
+		(at 199.39 52.07 0)
 		(fields_autoplaced yes)
 		(effects
@@
 		)
 		(property "Intersheetrefs" "${INTERSHEET_REFS}"
-			(at 217.2824 52.07 0)
+			(at 217.9174 52.07 0)
 			(effects
 				(font
@@
 		)
 	)
-	(global_label "transformer_S_N"
+	(global_label "transformer_S_P"
 		(shape output)
-		(at 198.755 41.91 0)
+		(at 199.39 41.91 0)
 		(fields_autoplaced yes)
 		(effects
@@
 		)
 		(property "Intersheetrefs" "${INTERSHEET_REFS}"
-			(at 217.2824 41.91 0)
+			(at 217.8569 41.91 0)
 			(effects
 				(font
@@
 	)
 	(symbol
-		(lib_id "Transformer:TEZ2.0-D-1")
-		(at 193.675 46.99 0)
-		(unit 1)
-		(exclude_from_sim no)
-		(in_bom yes)
-		(on_board yes)
-		(dnp no)
-		(property "Reference" "TR1"
-			(at 193.675 39.624 0)
-			(effects
-				(font
-					(size 1.27 1.27)
-				)
-			)
-		)
-		(property "Value" "Our Transformer"
-			(at 193.675 54.102 0)
-			(effects
-				(font
-					(size 1.27 1.27)
-				)
-			)
-		)
-		(property "Footprint" "Transformer_THT:Transformer_Breve_TEZ-28x33"
-			(at 193.675 55.88 0)
-			(effects
-				(font
-					(size 1.27 1.27)
-					(italic yes)
-				)
-				(hide yes)
-			)
-		)
-		(property "Datasheet" "http://www.breve.pl/pdf/ANG/TEZ_ang.pdf"
-			(at 193.675 46.99 0)
-			(effects
-				(font
-					(size 1.27 1.27)
-				)
-				(hide yes)
-			)
-		)
-		(property "Description" "TEZ2.0/D/x, 2VA, Single Secondary, Cast Resin Transformer, PCB"
-			(at 193.675 46.99 0)
-			(effects
-				(font
-					(size 1.27 1.27)
-				)
-				(hide yes)
-			)
-		)
-		(pin "5"
-		)
-		(pin "7"
-		)
-		(pin "9"
-		)
-		(pin "1"
-		)
-		(instances
-			(project ""
-				(path "/9378b4ad-d284-4009-8071-4a136b44f336"
-					(reference "TR1")
-					(unit 1)
-				)
-			)
-		)
-	)
-	(symbol
 		(lib_id "oscar:ISOUSB111DWXR")
 		(at 165.1 88.9 0)
@@
 	(symbol
 		(lib_id "Device:C")
-		(at 184.785 41.91 90)
+		(at 185.42 41.91 90)
 		(unit 1)
 		(exclude_from_sim no)
@@
 		(dnp no)
 		(property "Reference" "C29"
-			(at 184.785 45.466 90)
+			(at 185.42 45.466 90)
 			(effects
 				(font
@@
 		)
 		(property "Value" "C"
-			(at 184.785 38.354 90)
+			(at 185.42 38.354 90)
 			(effects
 				(font
@@
 		)
 		(property "Footprint" ""
-			(at 188.595 40.9448 0)
+			(at 189.23 40.9448 0)
 			(effects
 				(font
@@
 		)
 		(property "Datasheet" "~"
-			(at 184.785 41.91 0)
+			(at 185.42 41.91 0)
 			(effects
 				(font
@@
 		)
 		(property "Description" "Unpolarized capacitor"
-			(at 184.785 41.91 0)
+			(at 185.42 41.91 0)
 			(effects
 				(font
@@
 					(unit 1)
 				)
+			)
+		)
+	)
+	(symbol
+		(lib_id "Transformer:ED8_4")
+		(at 194.31 46.99 0)
+		(unit 1)
+		(exclude_from_sim no)
+		(in_bom yes)
+		(on_board yes)
+		(dnp no)
+		(property "Reference" "T1"
+			(at 194.31 36.83 0)
+			(effects
+				(font
+					(size 1.27 1.27)
+				)
+			)
+		)
+		(property "Value" "MAIN TRANSFORMER"
+			(at 194.31 38.862 0)
+			(effects
+				(font
+					(size 1.27 1.27)
+				)
+			)
+		)
+		(property "Footprint" "oscar:TRANSFORMER_PQ_PSFB"
+			(at 194.31 58.42 0)
+			(effects
+				(font
+					(size 1.27 1.27)
+				)
+				(hide yes)
+			)
+		)
+		(property "Datasheet" "https://gitlab.com/kicad/libraries/kicad-footprints/-/merge_requests/3626"
+			(at 194.31 60.96 0)
+			(effects
+				(font
+					(size 1.27 1.27)
+				)
+				(hide yes)
+			)
+		)
+		(property "Description" "600:600 Impedance Permalloy Core 1:1 Isolated Audio Transformer"
+			(at 194.31 55.88 0)
+			(effects
+				(font
+					(size 1.27 1.27)
+				)
+				(hide yes)
+			)
+		)
+		(pin "3"
+		)
+		(pin "1"
+		)
+		(pin "2"
+		)
+		(pin "4"
+		)
+		(instances
+			(project ""
+				(path "/9378b4ad-d284-4009-8071-4a136b44f336"
+					(reference "T1")
+					(unit 1)
+				)

Commit message: MCU conections
Connections:
- net CTRLA_H: now also U1.29 (PB15); no longer U1.31 (PA9)
- net CTRLA_L: now also U1.28 (PB14); no longer U1.30 (PA8)
- net I_IN_SENSE: now also U1.31 (PA9); no longer U1.16 (PB0)
- net I_OUT_SENSE: now also U1.16 (PB0); no longer U1.9 (PA1)
- net LED_FAULT_BATTERY: now also U1.14 (PA6); no longer U1.42 (PB5)
- net LED_FAULT_MCU: now also U1.13 (PA5); no longer U1.41 (PB4)
- net LED_MCU_ON: now also U1.10 (PA2); no longer U1.17 (PB1)
- net LED_OK: now also U1.11 (PA3); no longer U1.18 (PB2)
- net LED_STATUS: now also U1.12 (PA4); no longer U1.40 (PB3)
- net SSR: now also U1.8 (PA0); no longer U1.43 (PB6)
- net VDC_P_SENSE: now also U1.5 (PF0); no longer U1.8 (PA0)
- net VDC_S_SENSE: now also U1.6 (PF1); no longer U1.28 (PB14)
- net V_BAT_FLAG: now also U1.9 (PA1); no longer U1.29 (PB15)
- no-connect marks 24 -> 14
